File: pcb_ruler.kicad_pcb (KiCad board)
At the start: 2 copper layers, 304.8 x 25.4 mm, 1 part

Commit message: Added some logos to PCB
Other:
- board text added: "WELMEK"

Commit message: Added Mitra
Routing:
- net dummy: vias 0 -> 1
- net (no net): vias 1 -> 0
- added copper zone on B.Cu, net dummy
- added copper zone on F.Cu, net dummy
- removed copper zone on F.Cu, net (none)
Other:
- board text added: "Couvre-plancher RM SENC (514) 377-6324"

Commit message: Added Chalifoux, ProMach
Other:
- board text added: "EAU DE SOURCE NATURELLE"
- board text added: "amaro"
