File: pcb_ruler.kicad_pcb (KiCad board)
At the start: 2 copper layers, 304.8 x 25.4 mm, 1 part

Commit message: Done; ready for OnBoard
Routing:
- net dummy: vias 1 -> 0
- removed copper zone on B.Cu, net dummy
Other:
- board text added: "7605"
- board text added: "v1"

Commit message: v2025
Other:
- board text added: "ARGENT"
- board text added: "BRONZE"
- board text added: "DIAMANT"
- board text added: "MERCI À NOS COMMANDITAIRES 2024-2025:"
- board text added: "OR"
- board text added: "PLATINE"
- board text added: "Scorpion"
- board text removed: "Couvre-plancher RM SENC (514) 377-6324"
- board text removed: "MERCI À NOS COMMANDITAIRES:"
- board text removed: "v1"
